File: pcb.kicad_pcb (KiCad board)
At the start: 2 copper layers, 247.4 x 96.5 mm, 217 parts, among them J0 USB_mini_micro_B, P1 CONN_3X2, P2 CONN_4, SW1.1 Backtick, SW1.10 9, SW1.11 0, SW1.12 -, SW1.13 =, SW1.2 1, SW1.3 2, SW1.4 3, SW1.5 4, SW1.6 5, SW1.7 6, SW1.8 7, SW1.9 8, SW2A1 Tab, SW2A10 I, SW2A11 O, SW2A12 P, SW2A13 /, SW2A2 Q, SW2A3 W, SW2A4 E, SW2A5 R, SW2A6 T, SW2A8 Y, SW2A9 U, SW2B1 Tab, SW2B10 I, SW2B11 O, SW2B12 P, SW2B13 /, SW2B2 Q, SW2B3 W, SW2B4 E, SW2B5 R, SW2B6 T, SW2B7 Y, SW2B8 Y, SW2B9 U, SW3A1 Bksp, SW3A10 K, SW3A11 L, SW3A12 ;, SW3A13 Enter, SW3A2 A, SW3A3 S, SW3A4 D, SW3A5 F, SW3A6 G, SW3A8 H, SW3A9 J, SW3B1 Bksp, SW3B10 K, SW3B11 L, SW3B12 ;, SW3B13 Enter, SW3B2 A, SW3B3 S, SW3B4 D, SW3B5 F, SW3B6 G, SW3B7 H, SW3B8 H, SW3B9 J, SW4.7 Fn, SW4A1 LShift, SW4A10 ,, SW4A11 ., SW4A13 RShift, SW4A3 Z, SW4A4 X, SW4A5 C, SW4A6 V, SW4A8 N, SW4A9 M, SW4B1 LShift, SW4B10 ,, SW4B11 .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

Commit message: Added a bunch of additional switches for layouts
Parts:
- added D4.7: D, Diodes_SMD:D_SOD-323_HandSoldering, B.Cu at (195.3, 159.5)
- added D5.3: D, Diodes_SMD:D_SOD-323_HandSoldering, B.Cu at (119.1, 178.6)
- added D5.7: D, Diodes_SMD:D_SOD-323_HandSoldering, B.Cu at (204.8, 178.6)
- added SW4B7: H, footprints:MX_100_Plate, F.Cu at (200.0, 157.2)
- added SW5C1: LCtrl, footprints:MX_100_Plate, F.Cu at (85.7, 176.2)
- added SW5C2: LGUI, footprints:MX_100_Plate, F.Cu at (104.8, 176.2)
- added SW5C3: 1, footprints:MX_100_Plate, F.Cu at (123.8, 176.2)
- added SW5C4: LAlt, footprints:MX_100_Plate, F.Cu at (142.9, 176.2)
- added SW5C5: Fn, footprints:MX_200_Plate, F.Cu at (171.4, 176.2)
- added SW5C7: Fn, footprints:MX_200_Plate, F.Cu at (209.6, 176.2)
- added SW5C9: 1, footprints:MX_100_Plate, F.Cu at (238.1, 176.2)
- moved D5.2 21.7 mm to (100.0, 178.6), turned to 270 degrees
- moved D2.2 17.8 mm to (100.0, 121.4), turned to 270 degrees
- moved D3.2 17.8 mm to (100.0, 140.5), turned to 270 degrees
- moved D2.3 17.8 mm to (119.1, 121.4), turned to 270 degrees
- moved D3.3 17.8 mm to (119.1, 140.5), turned to 270 degrees
- moved D5.12 17.8 mm to (281.0, 178.6), turned to 270 degrees
- moved D4.13 17.8 mm to (300.0, 159.5), turned to 270 degrees
- moved D4.3 17.5 mm to (119.1, 159.5), turned to 270 degrees
- moved D4.1 17.5 mm to (81.0, 159.5), turned to 270 degrees
- moved D4.2 17.5 mm to (100.0, 159.5), turned to 270 degrees
- moved D5.10 17.1 mm to (252.4, 178.6), turned to 270 degrees
- moved D5.13 17.0 mm to (304.8, 178.6), turned to 270 degrees
- moved D5.1 17.0 mm to (81.0, 178.6), turned to 270 degrees
- moved D1 15.6 mm to (71.4, 95.2)
- moved D2.1 13.2 mm to (81.0, 121.4), turned to 270 degrees
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- renumbered D4.7 to D5.5, D5.7 to D5.9, SW4.7 to SW5A5, SW5A7 to SW5A9, SW5B7 to SW5B9
Connections:
- D5.5 pad 2: /matrix/Col7 -> Net-(D5.5-Pad2)
- D5.9 pad 2: /matrix/Col7 -> Net-(D5.9-Pad2)
- SW5A5 pad 1: /matrix/Row4 -> /matrix/Row5
Routing:
- net /matrix/Row3: track 0.00 -> 228.6 mm
- net /matrix/Col4: track 0.00 -> 91.0 mm
- net /matrix/Row5: track 230.4 -> 140.5 mm
- net /matrix/Col2: track 0.00 -> 87.9 mm
- net /matrix/Col3: track 0.00 -> 82.7 mm
- net /matrix/Col6: track 0.00 -> 68.8 mm
- net /matrix/Col7: track 0.00 -> 62.1 mm
- net /matrix/Col5: track 0.00 -> 61.6 mm
- net /matrix/Row4: track 239.7 -> 195.3 mm
- net Net-(D4.8-Pad1): track 14.1 -> 0.00 mm
- net Net-(D4.12-Pad1): track 14.1 -> 0.00 mm
- net Net-(D4.1-Pad1): track 14.0 -> 0.00 mm
- net Net-(D4.6-Pad1): track 14.0 -> 0.00 mm
- net Net-(D4.5-Pad1): track 14.0 -> 0.00 mm
- net Net-(D4.11-Pad1): track 14.0 -> 0.00 mm
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Other:
- board text added: "1"
- board text added: "1.25"
- board text added: "1.5"
- board text added: "2"
- board text added: "2.25"
- board text added: "2.75"

Commit message: All switch columns wired.
Wired all switches in a column together and dropped the 10 existing
WS2812Bs in place.  Need to connect everything to controller.
Parts:
- SW4A1, SW4A13, SW5C5, SW5C7: footprint footprints:MX_200_Plate -> footprints:MX_200_Plate_NoStabHoles
- SW5A5: footprint footprints:MX_225_Plate -> footprints:MX_225_Plate_NoStabHoles
- SW5A9, SW5B9: footprint footprints:MX_275_Plate -> footprints:MX_275_Plate_NoStabHoles
- moved LED1 258.3 mm to (292.9, 166.7), turned to 0 degrees
- moved LED2 224.5 mm to (254.8, 166.7), turned to 0 degrees
- moved LED10 221.2 mm to (214.3, 109.5), turned to 180 degrees
- moved C3 208.0 mm to (178.8, 180.0), turned to 270 degrees
- moved C2 199.6 mm to (181.4, 180.0), turned to 270 degrees
- moved OSC0 198.2 mm to (180.1, 175.6), turned to 180 degrees
- moved LED3 198.0 mm to (214.3, 166.7), turned to 0 degrees
- moved LED9 181.1 mm to (176.2, 109.5), turned to 180 degrees
- moved C6 179.3 mm to (183.9, 176.7), turned to 90 degrees
- moved C5 178.4 mm to (190.5, 183.3), turned to 180 degrees
- moved R3 177.9 mm to (183.9, 180.2), turned to 270 degrees
- moved C7 175.6 mm to (185.7, 161.9)
- moved R4 175.3 mm to (195.3, 163.2), turned to 0 degrees
- moved LED4 174.5 mm to (176.2, 166.7), turned to 0 degrees
- moved C4 167.3 mm to (199.1, 183.3), turned to 0 degrees
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Connections:
- D5.5 pad 2: Net-(D5.5-Pad2) -> /matrix/Col5
- D5.9 pad 2: Net-(D5.9-Pad2) -> /matrix/Col9
- U1 pad 20: /matrix/Col13 -> Net-(U1-Pad20)
- U1 pad 25: /matrix/Col7 -> /matrix/Row5
- U1 pad 26: /matrix/Col5 -> Net-(U1-Pad26)
- U1 pad 27: /matrix/Col3 -> Net-(U1-Pad27)
- U1 pad 28: /matrix/Row3 -> Net-(U1-Pad28)
- U1 pad 29: /matrix/Row5 -> /matrix/Col13
- U1 pad 30: /matrix/Row4 -> /matrix/Col12
- U1 pad 31: /matrix/Row1 -> /matrix/Col6
- U1 pad 32: /matrix/Row2 -> /matrix/Col7
- U1 pad 36: /matrix/Col1 -> Net-(U1-Pad36)
- U1 pad 37: /matrix/Col12 -> Net-(U1-Pad37)
- U1 pad 38: /matrix/Col10 -> Net-(U1-Pad38)
- U1 pad 39: /matrix/Col8 -> Net-(U1-Pad39)
- U1 pad 40: /matrix/Col6 -> Net-(U1-Pad40)
- U1 pad 41: /matrix/Col4 -> Net-(U1-Pad41)
Routing:
- net /matrix/Col13: track 0.00 -> 191.8 mm, vias 0 -> 2
- net /matrix/Col12: track 0.00 -> 177.1 mm, vias 0 -> 2
- net /underglow/Din: track 0.00 -> 127.4 mm, vias 0 -> 2
- net Net-(R1-Pad1): track 4.43 -> 118.4 mm, vias 0 -> 1
- net Net-(R2-Pad1): track 3.41 -> 116.5 mm, vias 0 -> 1
- net /matrix/Row5: track 140.5 -> 231.8 mm, vias 0 -> 1
- net Net-(LED6-Pad2): track 0.00 -> 83.7 mm, vias 0 -> 4
- net /matrix/Col10: track 0.00 -> 81.1 mm
- net /matrix/Col9: track 0.00 -> 80.5 mm
- net /matrix/Col11: track 0.00 -> 80.5 mm
- net /matrix/Col1: track 0.00 -> 79.0 mm
- net VCC: track 9.45 -> 75.7 mm, vias 0 -> 5
- net /matrix/Col8: track 0.00 -> 61.4 mm
- net /microcontroller/nRST: track 0.00 -> 48.7 mm, vias 0 -> 2
- net Net-(LED4-Pad2): track 0.00 -> 38.6 mm, vias 0 -> 2
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