File: pcb.kicad_pcb (KiCad board)
At the start: 2 copper layers, 247.4 x 97.8 mm, 194 parts, among them J0 USB_mini_micro_B, P1 CONN_01X06, P2 CONN_01X04, P3 CONN_01X03, P4 CONN_01X02, SW1.1 Backtick, SW1.10 9, SW1.11 0, SW1.12 -, SW1.13 =, SW1.2 1, SW1.3 2, SW1.4 3, SW1.5 4, SW1.6 5, SW1.7 6, SW1.8 7, SW1.9 8, SW2.1 Tab, SW2.10 I, SW2.11 O, SW2.12 P, SW2.13 /, SW2.2 Q, SW2.3 W, SW2.4 E, SW2.5 R, SW2.6 T, SW2.8 Y, SW2.9 U, SW3.1 Bksp, SW3.10 K, SW3.11 L, SW3.12 ;, SW3.13 Enter, SW3.2 A, SW3.3 S, SW3.4 D, SW3.5 F, SW3.6 G, SW3.8 H, SW3.9 J, SW4.10 ,, SW4.11 ., SW4.12 ., SW4.2 Z, SW4.3 Z, SW4.4 X, SW4.5 C, SW4.6 V, SW4.7 H, SW4.8 N, SW4.9 M, SW4A1 LShift, SW4A13 RShift, SW4B1 LShift, SW4B13 RShift, SW5A1 1.5, SW5A10 1.5, SW5A12 1.5, SW5A13 1.5, SW5A2 LGUI, SW5A4 LAlt, SW5A7 2.25, SW5A9 2.75, SW5B1 LCtrl, SW5B10 1, SW5B11 1, SW5B12 1, SW5B13 1, SW5B2 LGUI, SW5B3 1, SW5B4 LAlt, SW5B7 2.75, SW5B9 2.25, SW5C5 1.5, SW5C7 2/3, SW5C9 1.5, SW5D5 1, SW5D9 1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

Commit message: Updated USB footprint and added mounting holes
Updated mini USB to use included footprint.
Added two new mounting holes under bottom row of board.
Parts:
- added Hole4: M2, footprints:Mount_M2_Oval_NP, F.Cu at (97.6, 183.4)
- added Hole7: M2, footprints:Mount_M2_Oval_NP, F.Cu at (302.4, 183.4)
- J0: footprint keyboard_parts:USB_miniB_hirose_5S8 -> footprints:USB_miniB_hirose_5S8
- SW4.2: value Z -> ISO
- renumbered Hole4 to Hole5, Hole5 to Hole6
Changed lines of the file:
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@@
     (tracks 1353)
     (zones 0)
-    (modules 194)
+    (modules 196)
     (nets 113)
   )
@@
   )
   (module footprints:Mount_M2_Oval_NP (layer F.Cu)
-    (at 152.4 183.35625)
+    (at 97.63125 183.35625)
     (descr "Mounting Hole 2.2mm, M2")
     (tags "mounting hole 2.2mm m2")
@@
   )
   (module footprints:Mount_M2_Oval_NP (layer F.Cu)
-    (at 247.65 183.35625)
+    (at 302.41875 183.35625)
+    (descr "Mounting Hole 2.2mm, M2")
+    (tags "mounting hole 2.2mm m2")
+    (fp_text reference Hole7 (at 0 -3.2) (layer F.SilkS) hide
+      (effects (font (size 1 1) (thickness 0.15)))
+    )
+    (fp_text value M2 (at 0 3.2) (layer F.Fab)
+      (effects (font (size 1 1) (thickness 0.15)))
+    )
+    (fp_circle (center 0 0) (end 2.2 0) (layer Cmts.User) (width 0.15))
+    (fp_circle (center 0 0) (end 2.45 0) (layer F.CrtYd) (width 0.05))
+    (pad "" np_thru_hole oval (at 0 0) (size 4.6 2.5) (drill oval 4.6 2.5) (layers *.Cu *.Mask))
+  )
+  (module footprints:Mount_M2_Oval_NP (layer F.Cu)
+    (at 152.4 183.35625)
     (descr "Mounting Hole 2.2mm, M2")
     (tags "mounting hole 2.2mm m2")
@@
   )
   (module footprints:Mount_M2_Oval_NP (layer F.Cu)
+    (at 247.65 183.35625)
+    (descr "Mounting Hole 2.2mm, M2")
+    (tags "mounting hole 2.2mm m2")
+    (fp_text reference Hole6 (at 0 -3.2) (layer F.SilkS) hide
+      (effects (font (size 1 1) (thickness 0.15)))
+    )
+    (fp_text value M2 (at 0 3.2) (layer F.Fab)
+      (effects (font (size 1 1) (thickness 0.15)))
+    )
+    (fp_circle (center 0 0) (end 2.2 0) (layer Cmts.User) (width 0.15))
+    (fp_circle (center 0 0) (end 2.45 0) (layer F.CrtYd) (width 0.05))
+    (pad "" np_thru_hole oval (at 0 0) (size 4.6 2.5) (drill oval 4.6 2.5) (layers *.Cu *.Mask))
+  )
+  (module footprints:Mount_M2_Oval_NP (layer F.Cu)
     (at 319.0875 109.5375)
     (descr "Mounting Hole 2.2mm, M2")
@@
     )
   )
-  (module keyboard_parts:USB_miniB_hirose_5S8 (layer B.Cu)
-    (at 95.25 95.25)
-    (descr "USB miniB hirose UX60SC-MB-5S8")
-    (tags "USB miniB hirose through hole UX60SC-MB-5S8")
-    (fp_text reference J0 (at 0 -2.45) (layer B.SilkS) hide
-      (effects (font (size 0.8128 0.8128) (thickness 0.2032)) (justify mirror))
-    )
-    (fp_text value USB_mini_micro_B (at 0 -7.95) (layer Dwgs.User) hide
-      (effects (font (thickness 0.3048)))
-    )
-    (fp_line (start 3.85 0.4) (end 3.85 -6.1) (layer B.SilkS) (width 0.2))
-    (fp_line (start -3.85 0.4) (end -3.85 -6.1) (layer B.SilkS) (width 0.2))
-    (fp_line (start -3.85 0.4) (end 3.85 0.4) (layer B.SilkS) (width 0.2))
-    (fp_line (start -1 -6.1) (end 1 -6.1) (layer Dwgs.User) (width 0.2))
-    (fp_line (start -3.85 -6.6) (end -3.85 -5.7) (layer Dwgs.User) (width 0.2))
-    (fp_line (start 3.85 -6.6) (end 3.85 -5.7) (layer Dwgs.User) (width 0.2))
-    (fp_text user "PCB edge" (at -0.05 -5.35) (layer Dwgs.User) hide
-      (effects (font (size 0.5 0.5) (thickness 0.125)))
-    )
-    (fp_line (start -3.85 -6.6) (end 3.85 -6.6) (layer Dwgs.User) (width 0.2))
-    (pad 1 smd rect (at -1.6 0) (size 0.5 1.4) (layers B.Cu B.Paste B.Mask)
-      (net 102 "Net-(F1-Pad2)"))
-    (pad 2 smd rect (at -0.8 0) (size 0.5 1.4) (layers B.Cu B.Paste B.Mask)
-      (net 3 /microcontroller/USB_D-))
-    (pad 3 smd rect (at 0 0) (size 0.5 1.4) (layers B.Cu B.Paste B.Mask)
-      (net 4 /microcontroller/USB_D+))
-    (pad 4 smd rect (at 0.8 0) (size 0.5 1.4) (layers B.Cu B.Paste B.Mask)
-      (net 8 "Net-(J0-Pad4)"))
-    (pad 5 smd rect (at 1.6 0) (size 0.5 1.4) (layers B.Cu B.Paste B.Mask)
-      (net 2 GND))
-    (pad 6 thru_hole oval (at -3.65 -2.4) (size 1.3 3.8) (drill oval 0.7 3.2) (layers *.Cu *.Mask B.Paste)
-      (net 2 GND))
-    (pad 6 thru_hole oval (at 3.65 -2.4) (size 1.3 3.8) (drill oval 0.7 3.2) (layers *.Cu *.Mask B.Paste)
-      (net 2 GND))
-  )
   (module footprints:OSC_EpsonFA238_SMD (layer B.Cu)
     (at 118.364 127.381 315)
@@
       (effects (font (size 1 1) (thickness 0.2)) (justify mirror))
     )
-    (fp_text value Z (at 5.334 10.922) (layer B.SilkS) hide
+    (fp_text value ISO (at 5.334 10.922) (layer B.SilkS) hide
       (effects (font (thickness 0.3048)) (justify mirror))
     )
@@
     (pad "" np_thru_hole circle (at 0 0) (size 2.5 2.5) (drill 2.5) (layers *.Cu *.Mask))
   )
+  (module footprints:USB_miniB_hirose_5S8 (layer B.Cu)
+    (at 95.25 95.25)
+    (descr "USB miniB hirose UX60SC-MB-5S8")
+    (tags "USB miniB hirose through hole UX60SC-MB-5S8")
+    (fp_text reference J0 (at 0 -2.45) (layer B.SilkS) hide
+      (effects (font (size 0.8128 0.8128) (thickness 0.2032)) (justify mirror))
+    )
+    (fp_text value USB_mini_micro_B (at 0 -7.95) (layer Dwgs.User) hide
+      (effects (font (thickness 0.3048)))
+    )
+    (fp_line (start 3.85 0.4) (end 3.85 -6.1) (layer B.SilkS) (width 0.2))
+    (fp_line (start -3.85 0.4) (end -3.85 -6.1) (layer B.SilkS) (width 0.2))
+    (fp_line (start -3.85 0.4) (end 3.85 0.4) (layer B.SilkS) (width 0.2))
+    (fp_line (start -1 -6.1) (end 1 -6.1) (layer Dwgs.User) (width 0.2))
+    (fp_line (start -3.85 -6.6) (end -3.85 -5.7) (layer Dwgs.User) (width 0.2))
+    (fp_line (start 3.85 -6.6) (end 3.85 -5.7) (layer Dwgs.User) (width 0.2))
+    (fp_text user "PCB edge" (at -0.05 -5.35) (layer Dwgs.User) hide
+      (effects (font (size 0.5 0.5) (thickness 0.125)))
+    )
+    (fp_line (start -3.85 -6.6) (end 3.85 -6.6) (layer Dwgs.User) (width 0.2))
+    (pad 1 smd rect (at -1.6 0) (size 0.5 1.4) (layers B.Cu B.Paste B.Mask)
+      (net 102 "Net-(F1-Pad2)"))
+    (pad 2 smd rect (at -0.8 0) (size 0.5 1.4) (layers B.Cu B.Paste B.Mask)
+      (net 3 /microcontroller/USB_D-))
+    (pad 3 smd rect (at 0 0) (size 0.5 1.4) (layers B.Cu B.Paste B.Mask)
+      (net 4 /microcontroller/USB_D+))
+    (pad 4 smd rect (at 0.8 0) (size 0.5 1.4) (layers B.Cu B.Paste B.Mask)
+      (net 8 "Net-(J0-Pad4)"))
+    (pad 5 smd rect (at 1.6 0) (size 0.5 1.4) (layers B.Cu B.Paste B.Mask)
+      (net 2 GND))
+    (pad 6 thru_hole oval (at -3.65 -2.4) (size 1.3 3.8) (drill oval 0.7 3.2) (layers *.Cu *.Mask B.Paste)
+      (net 2 GND))
+    (pad 6 thru_hole oval (at 3.65 -2.4) (size 1.3 3.8) (drill oval 0.7 3.2) (layers *.Cu *.Mask B.Paste)
+      (net 2 GND))
+  )
   (gr_text A (at 159.131 184.404) (layer B.SilkS)

Commit message: Shifted locations of vias for WS2812/Capacitors and shifted a couple traces
Parts:
- added Stitch7: Via-0.6mm, footprints:Via-0.6mm, F.Cu at (243.2, 168.0)
- renumbered Stitch4 to Stitch5, Stitch4 to Stitch6
Routing:
- net VCC: track 698.0 -> 698.5 mm
