File: matrix.sch (KiCad schematic (older format))
At the start: 136 parts, among them SW1.1 Backtick, SW1.10 9, SW1.11 0, SW1.12 -, SW1.13 =, SW1.2 1, SW1.3 2, SW1.4 3, SW1.5 4, SW1.6 5, SW1.7 6, SW1.8 7, SW1.9 8, SW2A1 Tab, SW2A10 I, SW2A11 O, SW2A12 P, SW2A13 /, SW2A2 Q, SW2A3 W, SW2A4 E, SW2A5 R, SW2A6 T, SW2A8 Y, SW2A9 U, SW3A1 Bksp, SW3A10 K, SW3A11 L, SW3A12 ;, SW3A13 Enter, SW3A2 A, SW3A3 S, SW3A4 D, SW3A5 F, SW3A6 G, SW3A8 H, SW3A9 J, SW4.7 H, SW4A1 LShift, SW4A10 ,, SW4A11 ., SW4A13 RShift, SW4A3 Z, SW4A4 X, SW4A5 C, SW4A6 V, SW4A8 N, SW4A9 M, SW4C1 LShift, SW4C12 ., SW4C13 RShift, SW4C2 Z, SW5A1 1.5, SW5A10 1.5, SW5A12 1.5, SW5A13 1.5, SW5A2 LGUI, SW5A4 LAlt, SW5A7 2.25, SW5A9 2.75, SW5B7 2.75, SW5B9 2.25, SW5C1 LCtrl, SW5C10 1, SW5C11 1, SW5C12 1, SW5C13 1, SW5C2 LGUI, SW5C3 1, SW5C4 LAlt, SW5C5 1.5, SW5C7 2/3, SW5C9 1.5, SW5D5 1, SW5D9 1

Commit message: More progress on PCB
Cleaned up silkscreen layers
Updated switch footprints to remove front layer and hide reference on
back layer
Moved references on back layer
Moved bottom mounting holes on PCB
Cleaned up matrix schematic
Parts:
- SW4.2: renamed from SW4C2; value Z -> ISO
- renumbered SW2A1 to SW2.1, SW2A10 to SW2.10, SW2A11 to SW2.11, SW2A12 to SW2.12, SW2A13 to SW2.13, SW2A2 to SW2.2, SW2A3 to SW2.3, SW2A4 to SW2.4, SW2A5 to SW2.5, SW2A6 to SW2.6, SW2A8 to SW2.8, SW2A9 to SW2.9, SW3A1 to SW3.1, SW3A10 to SW3.10, SW3A11 to SW3.11, SW3A12 to SW3.12, SW3A13 to SW3.13, SW3A2 to SW3.2, SW3A3 to SW3.3, SW3A4 to SW3.4, SW3A5 to SW3.5, SW3A6 to SW3.6, SW3A8 to SW3.8, SW3A9 to SW3.9, SW4A10 to SW4.10, SW4A11 to SW4.11, SW4C12 to SW4.12, SW4A3 to SW4.3, SW4A4 to SW4.4, SW4A5 to SW4.5, SW4A6 to SW4.6, SW4A8 to SW4.8, SW4A9 to SW4.9, SW4C1 to SW4B1, SW4C13 to SW4B13, SW5C1 to SW5B1, SW5C10 to SW5B10, SW5C11 to SW5B11, SW5C12 to SW5B12, SW5C13 to SW5B13, SW5C2 to SW5B2, SW5C3 to SW5B3, SW5C4 to SW5B4
Connections:
- wire segments 91 -> 96
Other:
- moved on the sheet: D4.12, D4.2, D5.1, D5.10, D5.11, D5.12, D5.13, D5.2, D5.3, D5.4, D5.5, D5.7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
