File: pcb.sch (KiCad schematic (older format))
At the start: 7 parts, among them J0 USB_mini_micro_B, P1 CONN_02X03, P2 CONN_01X04, P3 CONN_01X03

Commit message: More progress on PCB
Cleaned up silkscreen layers
Updated switch footprints to remove front layer and hide reference on
back layer
Moved references on back layer
Moved bottom mounting holes on PCB
Cleaned up matrix schematic
Parts:
- removed D1: LED, footprints:LED_3mm_plusminus, symbol LED
- removed P1: CONN_02X03, Pin_Headers:Pin_Header_Straight_2x03_Pitch2.54mm, symbol CONN_02X03
- removed R5: 100, Resistors_SMD:R_0805, symbol R
- added P1: CONN_01X06, Pin_Headers:Pin_Header_Straight_1x06_Pitch2.54mm, symbol CONN_01X06
- added P4: CONN_01X02, Pin_Headers:Pin_Header_Straight_1x02_Pitch2.54mm, symbol CONN_01X02
Connections:
- net GND: now also P1.1 (P1), P4.1 (P1)
- net VCC: now also P1.2 (P2)
- net microcontroller/MISO: now also P1.3 (P3)
- net microcontroller/MOSI: now also P1.4 (P4)
- net microcontroller/SCK: now also P1.5 (P5)
- net microcontroller/nRST: now also P4.2 (P2)
- new net microcontroller/SS: P1.6 (P6)
Other:
- moved on the sheet: P2
Changed lines of the file:
@@
 L GND #PWR02
 U 1 1 587C6CDF
-P 3600 2950
-F 0 "#PWR02" H 3600 2950 30  0001 C CNN
-F 1 "GND" H 3600 2880 30  0001 C CNN
-F 2 "" H 3600 2950 60  0001 C CNN
-F 3 "" H 3600 2950 60  0001 C CNN
-	1    3600 2950
+P 3600 2850
+F 0 "#PWR02" H 3600 2850 30  0001 C CNN
+F 1 "GND" H 3600 2780 30  0001 C CNN
+F 2 "" H 3600 2850 60  0001 C CNN
+F 3 "" H 3600 2850 60  0001 C CNN
+	1    3600 2850
 	1    0    0    -1
 $EndComp
@@
 F20 "Row2" B R 5200 2450 60
 F21 "Row1" B R 5200 2350 60
-F22 "SCL" B L 4000 3150 60
-F23 "SDA" B L 4000 3250 60
-F24 "MISO" B L 4000 3850 60
-F25 "MOSI" B L 4000 4050 60
-F26 "SCK" B L 4000 3750 60
-F27 "nRST" I L 4000 4350 60
-F28 "LED" O L 4000 2350 60
-F29 "GLOW" O L 4000 4250 60
+F22 "SCL" B L 4000 4000 60
+F23 "SDA" B L 4000 4100 60
+F24 "MISO" B L 4000 3450 60
+F25 "MOSI" B L 4000 3350 60
+F26 "SCK" B L 4000 3250 60
+F27 "nRST" I L 4000 4200 60
+F28 "GLOW" O L 4000 4300 60
+F29 "SS" B L 4000 3150 60
 $EndSheet
 $Comp
 L GND #PWR03
 U 1 1 5908B3A5
-P 3250 3550
-F 0 "#PWR03" H 3250 3550 30  0001 C CNN
-F 1 "GND" H 3250 3480 30  0001 C CNN
-F 2 "" H 3250 3550 60  0001 C CNN
-F 3 "" H 3250 3550 60  0001 C CNN
-	1    3250 3550
+P 3300 4400
+F 0 "#PWR03" H 3300 4400 30  0001 C CNN
+F 1 "GND" H 3300 4330 30  0001 C CNN
+F 2 "" H 3300 4400 60  0001 C CNN
+F 3 "" H 3300 4400 60  0001 C CNN
+	1    3300 4400
 	1    0    0    -1
 $EndComp
@@
 L VCC #PWR04
 U 1 1 5908C1F6
-P 3250 3050
-F 0 "#PWR04" H 3250 3150 30  0001 C CNN
-F 1 "VCC" H 3250 3200 30  0000 C CNN
-F 2 "" H 3250 3050 60  0001 C CNN
-F 3 "" H 3250 3050 60  0001 C CNN
-	1    3250 3050
-	1    0    0    -1
+P 3300 4200
+F 0 "#PWR04" H 3300 4300 30  0001 C CNN
+F 1 "VCC" H 3300 4350 30  0000 C CNN
+F 2 "" H 3300 4200 60  0001 C CNN
+F 3 "" H 3300 4200 60  0001 C CNN
+	1    3300 4200
+	0    1    1    0
 $EndComp
 $Comp
 L GND #PWR05
 U 1 1 5908D619
-P 3300 4250
-F 0 "#PWR05" H 3300 4250 30  0001 C CNN
-F 1 "GND" H 3300 4180 30  0001 C CNN
-F 2 "" H 3300 4250 60  0001 C CNN
-F 3 "" H 3300 4250 60  0001 C CNN
-	1    3300 4250
+P 3250 3700
+F 0 "#PWR05" H 3250 3700 30  0001 C CNN
+F 1 "GND" H 3250 3630 30  0001 C CNN
+F 2 "" H 3250 3700 60  0001 C CNN
+F 3 "" H 3250 3700 60  0001 C CNN
+	1    3250 3700
 	1    0    0    -1
 $EndComp
@@
 L VCC #PWR06
 U 1 1 5908D7E5
-P 3500 3650
-F 0 "#PWR06" H 3500 3750 30  0001 C CNN
-F 1 "VCC" H 3500 3800 30  0000 C CNN
-F 2 "" H 3500 3650 60  0001 C CNN
-F 3 "" H 3500 3650 60  0001 C CNN
-	1    3500 3650
-	1    0    0    -1
-$EndComp
-$Comp
-L LED D1
-U 1 1 590FE2D7
-P 4900 1700
-F 0 "D1" H 4900 1800 50  0000 C CNN
-F 1 "LED" H 4900 1600 50  0000 C CNN
-F 2 "footprints:LED_3mm_plusminus" H 4900 1700 60  0001 C CNN
-F 3 "" H 4900 1700 60  0001 C CNN
-	1    4900 1700
-	-1   0    0    1
-$EndComp
-$Comp
-L GND #PWR07
-U 1 1 590FFDFC
-P 5200 1800
-F 0 "#PWR07" H 5200 1800 30  0001 C CNN
-F 1 "GND" H 5200 1730 30  0001 C CNN
-F 2 "" H 5200 1800 60  0001 C CNN
-F 3 "" H 5200 1800 60  0001 C CNN
-	1    5200 1800
-	1    0    0    -1
-$EndComp
-$Comp
-L R R5
-U 1 1 591032AE
-P 4350 1700
-F 0 "R5" V 4430 1700 50  0000 C CNN
-F 1 "100" V 4350 1700 50  0000 C CNN
-F 2 "Resistors_SMD:R_0805" H 4350 1700 60  0001 C CNN
-F 3 "" H 4350 1700 60  0001 C CNN
-	1    4350 1700
+P 3300 3550
+F 0 "#PWR06" H 3300 3650 30  0001 C CNN
+F 1 "VCC" H 3300 3700 30  0000 C CNN
+F 2 "" H 3300 3550 60  0001 C CNN
+F 3 "" H 3300 3550 60  0001 C CNN
+	1    3300 3550
 	0    1    1    0
 $EndComp
@@
 Wire Wire Line
 	3350 2750 3600 2750
-Wire Wire Line
-	3600 2750 3600 2950
 Wire Wire Line
 	3350 2850 3600 2850
@@
 	6700 2450 5200 2450
 Wire Wire Line
-	3150 3150 4000 3150
-Wire Wire Line
-	3150 3450 3250 3450
-Wire Wire Line
-	3250 3450 3250 3550
-Wire Wire Line
-	3250 3050 3250 3350
-Wire Wire Line
-	4000 4050 3200 4050
-Wire Wire Line
-	3300 4250 3300 4150
-Wire Wire Line
-	3300 4150 3200 4150
-Wire Wire Line
-	3200 3950 3500 3950
-Wire Wire Line
-	3500 3950 3500 3650
-Wire Wire Line
-	4000 2350 3850 2350
-Wire Wire Line
-	5200 1700 5200 1800
-Wire Wire Line
-	3850 2350 3850 1700
-Wire Wire Line
-	3850 1700 4200 1700
-Wire Wire Line
-	4500 1700 4700 1700
-Wire Wire Line
-	5100 1700 5200 1700
+	3150 4000 4000 4000
+Wire Wire Line
+	3150 4300 3300 4300
+Wire Wire Line
+	3300 4300 3300 4400
 $Sheet
 S 4000 4800 1200 1850
@@
 Wire Wire Line
 	3150 4900 4000 4900
-Wire Wire Line
-	4000 4250 3800 4250
-Wire Wire Line
-	3800 4250 3800 4900
-$Comp
-L CONN_02X03 P1
-U 1 1 594B843A
-P 2950 4050
-F 0 "P1" H 2950 4250 50  0000 C CNN
-F 1 "CONN_02X03" H 2950 3850 50  0000 C CNN
-F 2 "Pin_Headers:Pin_Header_Straight_2x03_Pitch2.54mm" H 2950 2850 50  0001 C CNN
-F 3 "" H 2950 2850 50  0000 C CNN
-	1    2950 4050
-	1    0    0    -1
-$EndComp
 $Comp
 L CONN_01X04 P2
 U 1 1 594B85A5
-P 2950 3300
-F 0 "P2" H 2950 3550 50  0000 C CNN
-F 1 "CONN_01X04" V 3050 3300 50  0000 C CNN
-F 2 "Pin_Headers:Pin_Header_Straight_1x04_Pitch2.54mm" H 2950 3300 50  0001 C CNN
-F 3 "" H 2950 3300 50  0000 C CNN
-	1    2950 3300
+P 2950 4150
+F 0 "P2" H 2950 4400 50  0000 C CNN
+F 1 "CONN_01X04" V 3050 4150 50  0000 C CNN
+F 2 "Pin_Headers:Pin_Header_Straight_1x04_Pitch2.54mm" H 2950 4150 50  0001 C CNN
+F 3 "" H 2950 4150 50  0000 C CNN
+	1    2950 4150
 	-1   0    0    1
 $EndComp
@@
 $EndComp
 Wire Wire Line
-	2700 3950 2600 3950
-Wire Wire Line
-	2600 3950 2600 3850
-Connection ~ 2600 3850
-Wire Wire Line
-	2700 4050 2500 4050
-Wire Wire Line
-	2500 4050 2500 3750
-Connection ~ 2500 3750
-Wire Wire Line
-	2700 4150 2600 4150
-Wire Wire Line
-	2600 4150 2600 4350
-Connection ~ 2600 4350
-Wire Wire Line
-	2600 4350 4000 4350
-Wire Wire Line
-	2500 3750 4000 3750
-Wire Wire Line
-	2600 3850 4000 3850
-Connection ~ 3800 4900
-Wire Wire Line
 	3150 5000 3300 5000
 Wire Wire Line
@@
 	3300 5100 3300 5200
 $Comp
-L GND #PWR08
+L GND #PWR07
 U 1 1 594BD05A
 P 3300 5200
-F 0 "#PWR08" H 3300 5200 30  0001 C CNN
+F 0 "#PWR07" H 3300 5200 30  0001 C CNN
 F 1 "GND" H 3300 5130 30  0001 C CNN
 F 2 "" H 3300 5200 60  0001 C CNN
@@
 $EndComp
 $Comp
-L VCC #PWR09
+L VCC #PWR08
 U 1 1 594BD194
 P 3300 4800
-F 0 "#PWR09" H 3300 4900 30  0001 C CNN
+F 0 "#PWR08" H 3300 4900 30  0001 C CNN
 F 1 "VCC" H 3300 4950 30  0000 C CNN
 F 2 "" H 3300 4800 60  0001 C CNN
@@
 $EndComp
 Wire Wire Line
-	3250 3350 3150 3350
-Wire Wire Line
-	3150 3250 4000 3250
+	3300 4200 3150 4200
+Wire Wire Line
+	3150 4100 4000 4100
+Wire Wire Line
+	3600 2850 3600 2750
+Wire Wire Line
+	4000 4200 3800 4200
+Wire Wire Line
+	3800 4200 3800 4550
+Wire Wire Line
+	3800 4550 2600 4550
+Wire Wire Line
+	4000 4300 3900 4300
+Wire Wire Line
+	3900 4300 3900 4900
+Connection ~ 3900 4900
+$Comp
+L CONN_01X02 P4
+U 1 1 59529D24
+P 2400 4600
+F 0 "P4" H 2400 4750 50  0000 C CNN
+F 1 "CONN_01X02" V 2500 4600 50  0000 C CNN
+F 2 "Pin_Headers:Pin_Header_Straight_1x02_Pitch2.54mm" H 2400 4600 50  0001 C CNN
+F 3 "" H 2400 4600 50  0000 C CNN
+	1    2400 4600
+	-1   0    0    1
+$EndComp
+$Comp
+L GND #PWR09
+U 1 1 5952A2D6
+P 2700 4750
+F 0 "#PWR09" H 2700 4750 30  0001 C CNN
+F 1 "GND" H 2700 4680 30  0001 C CNN
+F 2 "" H 2700 4750 60  0001 C CNN
+F 3 "" H 2700 4750 60  0001 C CNN
+	1    2700 4750
+	1    0    0    -1
+$EndComp
+Wire Wire Line
+	2700 4750 2700 4650
+Wire Wire Line
+	2700 4650 2600 4650
+Wire Wire Line
+	4000 3450 3150 3450
+Wire Wire Line
+	4000 3350 3150 3350
+Wire Wire Line
+	4000 3250 3150 3250
+Wire Wire Line
+	4000 3150 3150 3150
+$Comp
+L CONN_01X06 P1
+U 1 1 59530B97
+P 2950 3400
+F 0 "P1" H 2950 3750 50  0000 C CNN
+F 1 "CONN_01X06" V 3050 3400 50  0000 C CNN
+F 2 "Pin_Headers:Pin_Header_Straight_1x06_Pitch2.54mm" H 2950 3400 50  0001 C CNN
+F 3 "" H 2950 3400 50  0000 C CNN
+	1    2950 3400
+	-1   0    0    1
+$EndComp
+Wire Wire Line
+	3150 3550 3300 3550
+Wire Wire Line
+	3250 3700 3250 3650
+Wire Wire Line
+	3250 3650 3150 3650
 $EndSCHEMATC

Commit message: Updated USB footprint and added mounting holes
Updated mini USB to use included footprint.
Added two new mounting holes under bottom row of board.
Parts:
- J0: footprint keyboard_parts:USB_miniB_hirose_5S8 -> footprints:USB_miniB_hirose_5S8
Changed lines of the file:
@@
 F 0 "J0" H 2800 2450 60  0000 C CNN
 F 1 "USB_mini_micro_B" H 3050 2750 60  0001 C CNN
-F 2 "keyboard_parts:USB_miniB_hirose_5S8" H 3150 2500 60  0001 C CNN
+F 2 "footprints:USB_miniB_hirose_5S8" H 3150 2500 60  0001 C CNN
 F 3 "" H 3150 2500 60  0000 C CNN
 	1    3200 2500
